File: _restore_backup_2026-06-25T14-05-50-874/DEV_BOARD.kicad_sch (KiCad schematic)
At the start: 34 parts, among them J1 USB_C_Receptacle_USB2.0_16P, J2 Conn_ARM_SWD_TagConnect_TC2030, U1 MSPM0G350x, U2 USBLC6-2SC6, U3 SPX3819M5-L-3-3, U4 CH340E, U5 LIS2DH, X1 8MHz

Commit message: Routing completed
Connections:
- net INT1: now also U1.36 (PB17/A1_4); no longer U1.22 (PB8)
- net INT2: now also U1.26 (PB16); no longer U1.23 (PB9)
- net UART0CTS: now also U4.5 (~{CTS}); no longer U4.4 (~{RTS})
- net UART0RTS: now also U4.4 (~{RTS}); no longer U4.5 (~{CTS})
Changed lines of the file:
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@@
+	)
+	(no_connect
+		(at 321.31 97.79)
 	)
 	(no_connect
@@
 	)
 	(no_connect
+		(at 321.31 102.87)
+	)
+	(no_connect
 		(at 273.05 73.66)
 	)
@@
 	)
 	(no_connect
-		(at 321.31 87.63)
-	)
-	(no_connect
 		(at 321.31 77.47)
 	)
@@
 	)
 	(no_connect
-		(at 321.31 85.09)
-	)
-	(no_connect
 		(at 273.05 81.28)
 	)
@@
 	(wire
 		(pts
-			(xy 179.07 118.11) (xy 179.07 124.46)
-		)
-		(stroke
-			(width 0)
-			(type default)
-		)
-	)
-	(wire
-		(pts
-			(xy 323.85 97.79) (xy 323.85 96.52)
-		)
-		(stroke
-			(width 0)
-			(type default)
-		)
-	)
-	(wire
-		(pts
 			(xy 217.17 107.95) (xy 260.35 107.95)
 		)
@@
 	(wire
 		(pts
-			(xy 172.72 105.41) (xy 162.56 105.41)
-		)
-		(stroke
-			(width 0)
-			(type default)
-		)
-	)
-	(wire
-		(pts
 			(xy 95.25 171.45) (xy 95.25 172.72)
 		)
@@
 	(wire
 		(pts
-			(xy 162.56 118.11) (xy 179.07 118.11)
-		)
-		(stroke
-			(width 0)
-			(type default)
-		)
-	)
-	(wire
-		(pts
 			(xy 62.23 67.31) (xy 72.39 67.31)
 		)
@@
 	(wire
 		(pts
+			(xy 162.56 105.41) (xy 184.15 105.41)
+		)
+		(stroke
+			(width 0)
+			(type default)
+		)
+	)
+	(wire
+		(pts
 			(xy 389.89 63.5) (xy 398.78 63.5)
 		)
@@
 	(wire
 		(pts
+			(xy 184.15 105.41) (xy 184.15 124.46)
+		)
+		(stroke
+			(width 0)
+			(type default)
+		)
+	)
+	(wire
+		(pts
 			(xy 72.39 90.17) (xy 72.39 91.44)
 		)
@@
 	(wire
 		(pts
-			(xy 179.07 124.46) (xy 217.17 124.46)
+			(xy 184.15 124.46) (xy 217.17 124.46)
 		)
 		(stroke
@@
 	(wire
 		(pts
-			(xy 321.31 102.87) (xy 323.85 102.87)
-		)
-		(stroke
-			(width 0)
-			(type default)
-		)
-	)
-	(wire
-		(pts
 			(xy 220.98 96.52) (xy 273.05 96.52)
 		)
@@
 	(wire
 		(pts
-			(xy 172.72 105.41) (xy 172.72 125.73)
-		)
-		(stroke
-			(width 0)
-			(type default)
-		)
-	)
-	(wire
-		(pts
 			(xy 363.22 64.77) (xy 363.22 66.04)
 		)
@@
 	(wire
 		(pts
+			(xy 172.72 118.11) (xy 162.56 118.11)
+		)
+		(stroke
+			(width 0)
+			(type default)
+		)
+	)
+	(wire
+		(pts
 			(xy 226.06 124.46) (xy 234.95 124.46)
 		)
@@
 	(wire
 		(pts
-			(xy 321.31 97.79) (xy 323.85 97.79)
-		)
-		(stroke
-			(width 0)
-			(type default)
-		)
-	)
-	(wire
-		(pts
 			(xy 264.16 82.55) (xy 264.16 86.36)
 		)
@@
 		(pts
 			(xy 63.5 77.47) (xy 81.28 77.47)
+		)
+		(stroke
+			(width 0)
+			(type default)
+		)
+	)
+	(wire
+		(pts
+			(xy 172.72 125.73) (xy 172.72 118.11)
 		)
 		(stroke
@@
 	(global_label "INT1"
 		(shape input)
-		(at 323.85 102.87 0)
+		(at 321.31 85.09 0)
 		(fields_autoplaced yes)
 		(effects
@@
 		)
 		(property "Intersheetrefs" "${INTERSHEET_REFS}"
-			(at 330.9476 102.87 0)
+			(at 328.4076 85.09 0)
 			(hide yes)
 			(show_name no)
@@
 	(global_label "INT2"
 		(shape input)
-		(at 323.85 96.52 0)
+		(at 321.31 87.63 0)
 		(fields_autoplaced yes)
 		(effects
@@
 		)
 		(property "Intersheetrefs" "${INTERSHEET_REFS}"
-			(at 330.9476 96.52 0)
+			(at 328.4076 87.63 0)
 			(hide yes)
 			(show_name no)
